File: FPGA.kicad_pcb (KiCad board)
At the start: 8 copper layers, 83 parts, among them IC1 MAX20029ATIF_V+, J1 Conn_02x07_Odd_Even, J10 Conn_01x03_Socket, J3 Conn_01x10_Socket, J4 Conn_01x10_Socket, Q1 2N7000, Q2 2N7000, Q3 2N7000, Q4 2N7000, U1 XC7A15T-FTG256, U2 REF3012, X1 ECS-2520MV-160-CN-TR

Commit message: continued PCB design
Parts:
- moved J10 23.4 mm to (101.0, 78.0), turned to -90 degrees
- moved C10 10.8 mm to (175.7, 64.8)
- moved C32 10.8 mm to (184.6, 64.3)
- moved C45 10.8 mm to (167.0, 60.5)
- moved C46 10.8 mm to (161.0, 64.5)
- moved C47 10.8 mm to (169.1, 69.8)
- moved C5 10.8 mm to (169.5, 64.5)
- moved C31 10.8 mm to (194.5, 61.7)
- moved C33 10.8 mm to (191.2, 62.8)
- moved C34 10.8 mm to (187.9, 64.0)
- moved C39 10.8 mm to (181.0, 59.3)
- moved C40 10.8 mm to (164.6, 71.3)
- moved C41 10.8 mm to (160.6, 71.8)
- moved C42 10.8 mm to (174.6, 68.9)
- moved C44 10.8 mm to (164.6, 65.2)
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Routing:
- net TMS: track 0.00 -> 0.64 mm, vias 0 -> 1
- net TDI: track 0.00 -> 0.64 mm, vias 0 -> 1
- net TCK: track 0.00 -> 0.64 mm, vias 0 -> 1
- net Net-(U1C-VREFP_0): track 0.00 -> 0.64 mm, vias 0 -> 1
- net Net-(U1C-PROGRAM_B_0): track 0.00 -> 0.64 mm, vias 0 -> 1
- net Net-(J4-Pin_9): track 0.00 -> 0.64 mm, vias 0 -> 1
- net Net-(J4-Pin_8): track 0.00 -> 0.64 mm, vias 0 -> 1
- net Net-(J4-Pin_5): track 0.00 -> 0.64 mm, vias 0 -> 1
- net Net-(J4-Pin_3): track 0.00 -> 0.64 mm, vias 0 -> 1
- net Net-(J4-Pin_2): track 0.00 -> 0.64 mm, vias 0 -> 1
- net Net-(J4-Pin_10): track 0.00 -> 0.64 mm, vias 0 -> 1
- net Net-(J4-Pin_1): track 0.00 -> 0.64 mm, vias 0 -> 1
- net Net-(J3-Pin_9): track 0.00 -> 0.64 mm, vias 0 -> 1
- net Net-(J3-Pin_8): track 0.00 -> 0.64 mm, vias 0 -> 1
- net Net-(J3-Pin_7): track 0.00 -> 0.64 mm, vias 0 -> 1
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- added copper zone on In3.Cu, net GND
- added copper zone on In6.Cu, net GND
Other:
- board outline added: 50 x 50 mm
