File: FPGA.kicad_pcb (KiCad board)
At the start: 8 copper layers, 50 x 50 mm, 83 parts, among them IC1 MAX20029ATIF_V+, J1 Conn_02x07_Odd_Even, J10 Conn_01x03_Socket, J3 Conn_01x10_Socket, J4 Conn_01x10_Socket, Q1 2N7000, Q2 2N7000, Q3 2N7000, Q4 2N7000, U1 XC7A15T-FTG256, U2 REF3012, X1 ECS-2520MV-160-CN-TR

Commit message: FINISHED :3
Parts:
- C14, C6, C9: moved to B.Cu
- C39, C40, C41, C42, C43, C44: moved to F.Cu
- C45, C46, C47, C48, C8: footprint Capacitor_SMD:C_0402_1005Metric -> Capacitor_SMD:C_0603_1608Metric
- moved C31 111.1 mm to (91.8, 103.8)
- moved C33 108.6 mm to (91.8, 106.5)
- moved C14 106.9 mm to (113.0, 114.0)
- moved C34 106.2 mm to (91.7, 109.0)
- moved C32 104.2 mm to (91.8, 111.5)
- moved C6 104.0 mm to (96.2, 97.8), turned to 90 degrees
- moved C9 98.3 mm to (107.8, 97.8), turned to 90 degrees
- moved R5 82.9 mm to (85.5, 87.2), turned to 180 degrees
- moved C39 81.9 mm to (103.2, 84.9), turned to 0 degrees
- moved C4 81.3 mm to (98.0, 98.0), turned to 90 degrees
- moved C42 80.3 mm to (95.5, 82.7)
- moved R4 78.7 mm to (85.5, 88.5), turned to 180 degrees
- moved C10 77.9 mm to (105.2, 98.0), turned to 90 degrees
- moved C8 77.3 mm to (110.5, 97.8), turned to 90 degrees
- moved C47 76.9 mm to (95.5, 92.2), turned to 90 degrees
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Routing:
- net 3.3V: track 33.2 -> 256.8 mm, vias 26 -> 29
- net GND: track 23.8 -> 152.6 mm, vias 33 -> 69
- net 1.8V: track 5.60 -> 100.1 mm, vias 6 -> 12
- net 1V: track 6.43 -> 97.9 mm, vias 9 -> 15
- net TDI: track 0.64 -> 87.5 mm, vias 1 -> 2
- net EN1: track 0.00 -> 73.6 mm, vias 0 -> 7
- net TMS: track 0.64 -> 69.5 mm, vias 1 -> 2
- net TCK: track 0.64 -> 64.9 mm, vias 1 -> 2
- net TDO: track 0.00 -> 59.3 mm, vias 0 -> 2
- net 1.2V: track 0.00 -> 57.0 mm, vias 0 -> 5
- net INIT_B: track 0.64 -> 39.4 mm, vias 1 -> 2
- net Net-(J3-Pin_1): track 0.64 -> 35.5 mm, vias 1 -> 2
- net EN3: track 0.00 -> 33.0 mm, vias 0 -> 3
- net Net-(J3-Pin_2): track 0.64 -> 33.0 mm, vias 1 -> 2
- net Net-(J4-Pin_5): track 0.64 -> 31.2 mm, vias 1 -> 2
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