File: _autosave-FPGA.kicad_pcb (KiCad board)
At the start: 8 copper layers, 50 x 50 mm, 83 parts, among them IC1 MAX20029ATIF_V+, J1 Conn_02x07_Odd_Even, J10 Conn_01x03_Socket, J3 Conn_01x10_Socket, J4 Conn_01x10_Socket, Q1 2N7000, Q2 2N7000, Q3 2N7000, Q4 2N7000, U1 XC7A15T-FTG256, U2 REF3012, X1 ECS-2520MV-160-CN-TR

Commit message: almost finished the rough placement, only some resistors and decoupling caps remain
Parts:
- moved C12 61.2 mm to (98.5, 105.5), turned to 90 degrees
- moved C3 60.4 mm to (102.0, 105.8), turned to -90 degrees
- moved C2 54.9 mm to (106.2, 110.0), turned to 0 degrees
- moved C7 52.4 mm to (102.0, 110.0), turned to 90 degrees
- moved C1 50.5 mm to (104.5, 108.2), turned to 0 degrees
- moved C13 48.0 mm to (106.2, 105.2), turned to 0 degrees
- moved R2 26.4 mm to (144.0, 102.0)
- moved C10 20.9 mm to (163.0, 48.2)
- moved C8 20.8 mm to (169.3, 46.8)
- moved C11 20.7 mm to (167.0, 50.2), turned to 0 degrees
- moved R1 19.4 mm to (148.0, 106.0)
- moved C45 16.6 mm to (165.0, 44.0)
- moved C15 15.7 mm to (139.5, 87.5), turned to 0 degrees
- moved C16 15.4 mm to (134.5, 91.2)
Routing:
- net 1.8V: track 5.60 -> 7.01 mm
