File: Power.kicad_sch (KiCad schematic)
At the start: 16 parts, among them J10 Conn_01x03_Socket, U1 XC7A15T-FTG256

Commit message: FINISHED :3
Parts:
- C8: footprint Capacitor_SMD:C_0402_1005Metric -> Capacitor_SMD:C_0603_1608Metric
Changed lines of the file:
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@@
       (effects (font (size 1.27 1.27)) (justify left))
     )
-    (property "Footprint" "Capacitor_SMD:C_0402_1005Metric" (at 110.1852 106.68 0)
+    (property "Footprint" "Capacitor_SMD:C_0603_1608Metric" (at 110.1852 106.68 0)
       (effects (font (size 1.27 1.27)) hide)
     )
