File: Power_Supply.kicad_sch (KiCad schematic)
At the start: 28 parts, among them IC1 MAX20029ATIF_V+, Q1 2N7000

Commit message: FINISHED :3
Parts:
- C45, C46, C47, C48: footprint Capacitor_SMD:C_0402_1005Metric -> Capacitor_SMD:C_0603_1608Metric
Changed lines of the file:
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@@
       (effects (font (size 1.27 1.27)) (justify left))
     )
-    (property "Footprint" "Capacitor_SMD:C_0402_1005Metric" (at 265.1252 123.19 0)
+    (property "Footprint" "Capacitor_SMD:C_0603_1608Metric" (at 265.1252 123.19 0)
       (effects (font (size 1.27 1.27)) hide)
     )
@@
       (effects (font (size 1.27 1.27)) (justify left))
     )
-    (property "Footprint" "Capacitor_SMD:C_0402_1005Metric" (at 265.1252 60.96 0)
+    (property "Footprint" "Capacitor_SMD:C_0603_1608Metric" (at 265.1252 60.96 0)
       (effects (font (size 1.27 1.27)) hide)
     )
@@
       (effects (font (size 1.27 1.27)) (justify left))
     )
-    (property "Footprint" "Capacitor_SMD:C_0402_1005Metric" (at 265.1252 148.59 0)
+    (property "Footprint" "Capacitor_SMD:C_0603_1608Metric" (at 265.1252 148.59 0)
       (effects (font (size 1.27 1.27)) hide)
     )
@@
       (effects (font (size 1.27 1.27)) (justify left))
     )
-    (property "Footprint" "Capacitor_SMD:C_0402_1005Metric" (at 265.1252 86.36 0)
-      (effects (font (size 1.27 1.27)) hide)
-    )
+    (property "Footprint" "Capacitor_SMD:C_0603_1608Metric" (at 265.1252 86.36 0)
+      (effects (font (size 1.27 1.27)) hide)
+    )
